File: SYS1.kicad_pcb (KiCad board)
At the start: 4 copper layers, 100 x 100 mm, 149 parts, among them J1 338069-8, J10 8-338069-8, J101 Conn_01x03_Pin, J2 Micro_SD_Card, J3 SIM8051-6-0-14-01-X-REVD, J4 Conn_01x04_Pin, J6 2169890001, J7 430450800, J9 338069-8, Q1 NPN, Q2 NPN, Q3 NPN, Q4 NPN, Q5 NPN, U1 STM32F103VETx, U2 M65, U3 RASPBERRY_PI_ZERO_2_W, U300 TMP117xxDRV, U301 MS5611-01BA, U302 L96-M33, U303 BME680, Y101 8MHz, Y102 32.768KHz

Commit message: Velike izmene PCB
Zavrsena mala spoljanja plocica
Preliminarni placement komponenti na velikoj plocici
Dodati logotipi ISP i ELE
Dodato potpise
Parts:
- removed R104: 1M, Resistor_SMD:R_1206_3216Metric_Pad1.30x1.75mm_HandSolder
- removed Y102: 32.768KHz, Crystal:Crystal_HC49-U_Vertical
- added G***: LOGO, Potpisi:Lena, F.Cu at (68.2, 99.5)
- added G***: LOGO, Potpisi:ISP, F.Cu at (61.0, 64.2)
- added G***: LOGO, Potpisi:Nikola, F.Cu at (60.5, 99.5)
- added G***: LOGO, Potpisi:Jovan, F.Cu at (76.0, 76.5)
- added G***: LOGO, Potpisi:Marijana, F.Cu at (60.0, 78.8)
- added G***: LOGO, Potpisi:ELE, F.Cu at (70.5, 64.0)
- added Y1: ABS25-32.768KHZ-T, Crystal:Crystal_SMD_Abracon_ABS25-4Pin_8.0x3.8mm, B.Cu at (93.3, 111.8)
- C102, C103: value 22pF -> 15pF; moved to B.Cu
- C104, C105: value 22pF -> 27pF; moved to B.Cu
- C106, C107, C108, C109, C110, C111, C112, C113, C114, C115, C116, C217, C218, C219, C221, C222, C302, C303, C304, C305, C306, C307, C308, C309, R1, R118, R119, R120, R121, R122, R2, R210, R211, R212, R213, R3, R307, R308, R4, TP11, TP12, TP13, TP14, TP17, TP18, TP19, TP20, TP26, TP27: moved to B.Cu
- Q1, Q2: moved to F.Cu
- Y101: footprint Crystal:Crystal_HC49-U_Vertical -> Crystal:Crystal_SMD_HC49-SD; moved to B.Cu
- moved R301 363.9 mm to (186.5, 59.8), turned to 90 degrees
- moved R4 354.6 mm to (178.2, 53.8), turned to -90 degrees
- moved C301 354.3 mm to (182.5, 57.0), turned to 90 degrees
- moved U300 353.7 mm to (186.5, 63.9), turned to 180 degrees
- moved JP301 352.7 mm to (186.4, 54.5), turned to 180 degrees
- moved R3 351.9 mm to (175.8, 53.8), turned to -90 degrees
- moved R2 349.3 mm to (173.2, 53.8), turned to -90 degrees
- moved R1 346.8 mm to (170.8, 53.8), turned to -90 degrees
- moved J1 339.2 mm to (175.0, 75.2)
- moved H5 321.5 mm to (175.0, 65.0)
- moved R308 321.4 mm to (139.6, 55.0), turned to -90 degrees
- moved C309 318.7 mm to (143.2, 61.0), turned to -90 degrees
- moved R307 317.5 mm to (136.3, 55.0), turned to -90 degrees
- moved D4 315.6 mm to (178.2, 53.7), turned to -90 degrees
- moved C308 314.8 mm to (139.9, 61.0), turned to -90 degrees
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Routing:
- net DIAG3_EXT: track 0.00 -> 20.5 mm
- net I2C_SDA_EXT: track 0.00 -> 20.5 mm
- net DIAG4_EXT: track 0.00 -> 19.8 mm
- net DIAG2_EXT: track 0.00 -> 19.6 mm
- net DIAG1_EXT: track 0.00 -> 18.9 mm
- net I2C_SCL_EXT: track 0.00 -> 18.6 mm
- net EXT_GND: track 0.00 -> 9.56 mm, vias 0 -> 4
- net Net-(JP301-C): track 0.00 -> 3.72 mm
- net Net-(U300-ADD0): track 0.00 -> 2.27 mm
- net EXT_+3.3V: track 0.00 -> 1.19 mm
- net Net-(D4-K): vias 0 -> 1
- net Net-(D3-K): vias 0 -> 1
- net Net-(D2-K): vias 0 -> 1
- net Net-(D1-K): vias 0 -> 1
- added copper zone on F.Cu, net EXT_+3.3V
- added copper zone on B.Cu, net EXT_GND
Other:
- board size 100 x 100 mm -> 140 x 100 mm
- board text added: "Aleksandar Lukic"
- board text added: "Created by:"
- board text added: "ELEKvadar 2.0"
- board text added: "SYS1"
- board text added: "SYS1 EXT"
- board text added: "SYS1 MAIN"
- board text added: "Stevan Golubovic"
